File: CellKeeper.kicad_sch (KiCad schematic)
At the start: 528 parts, among them J1 Screw_Terminal_01x04, J10 3.81P Screw Terminal, J11 USB_C_Receptacle_USB2.0_16P, J12 Conn_02x10_Odd_Even, J13 USB_C_Receptacle_USB2.0_16P, J14 OEM Shunt Connector, J15 Screw_Terminal_01x04, J16 Conn_01x03, J17 OEM HV Sense Connector, J18 7.62mm Pitch Screw Terminal, J19 USB_C_Receptacle_USB2.0_16P, J2 Screw_Terminal_01x01, J20 OEM Connector, J21 3.81P Screw Terminal, J22 Conn_02x10_Odd_Even, J23 OEM Connector, J24 3.81P Screw Terminal, J3 Screw_Terminal_01x04, J4 8P8C_LED_Shielded_x2, J5 8P8C_LED_Shielded_x2, J6 OEM Connector, J7 Screw_Terminal_01x04, J8 Conn_01x03, J9 USB_C_Receptacle_USB2.0_16P, K1 Link Positive, K10 Inverter, K2 Link Negative, K3 FC Positive, K4 FC Negative, K5 Inverter, K6 Link Positive, K7 Link Negative, K8 FC Negative, K9 FC Positive, Q1 BSC0805LS, Q2 BSC0805LS, Q3 BSC0805LS, Q4 BSC0805LS, SW1 TS-1187A-B-A-B, SW2 TS-1187A-B-A-B, SW3 TS-1187A-B-A-B, SW4 TS-1187A-B-A-B, U1 UCC27524DR, U10 ISO1050DUB, U11 UCC27524DR, U12 LTV-217-B-G, U13 LTV-217-B-G, U14 RP2354B, U15 F0505S-1WR3, U16 ISO1540, U17 INA228, U18 ADS1115, U19 ADS1115, U20 RP2354B, U21 SP3485EN-L/TR, U22 AM26LV32EIDR, U23 SP3485EN-L/TR, U24 AM26LV32EIDR, U25 TLV1117LV33DCYR, U26 TLV1117LV33DCYR, U3 TPS5430DDAR, U4 F0505S-1WR3, U5 ISO1050DUB, U6 LTV-217-B-G, U7 LTV-217-B-G, U8 LTV-217-B-G, U9 LTV-217-B-G, Y1 ABM8-272-T3, Y2 ABM8-272-T3

Commit message: Rev1.1: USB VBUS sense on GPIO3, revision strap, shunt 3V3 cap
- USB VBUS detect for both MCUs: 3.3k from each connector's VBUS to GPIO3
  (pin 80) and 5.1k to GND (controller R78/R153, Supervisor R155/R154), also
  brought out on J12/J22 pin 2.
- Revision strap on GPIO47: R75 10k to 3V3, R76 1k to GND (reads as Rev1.1).
- C116 10uF on the isolated shunt 3V3; C57 removed.
- Test points: GPIO1-3 removed, GPIO44-46 added.
Parts:
- removed GPIO3: TP, CellKeeper_Local:BMS_Library__TestPoint_THTPad_D1.5mm_Drill1.0mm, symbol CellKeeper_Local:Connector__TestPoint_Small
- added GPIO46: TP, CellKeeper_Local:BMS_Library__TestPoint_THTPad_D1.5mm_Drill1.0mm, symbol CellKeeper_Local:Connector__TestPoint_Small
- added R153, R154: 5.1k, CellKeeper_Local:Resistor_SMD__R_0603_1608Metric, symbol CellKeeper_Local:Device__R_Small
- added R155, R78: 3.3k, CellKeeper_Local:Resistor_SMD__R_0402_1005Metric, symbol CellKeeper_Local:Device__R_Small
- R75: value 47k -> 10k; JLCPCB Part # C25819 -> C25804; now fitted
- R76: value 0r -> 1k; JLCPCB Part # C21189 -> C21190
- renumbered GPIO1 to GPIO44, GPIO2 to GPIO45
Connections:
- net GND: now also R153.2, R154.2
- net GPIO46_ADC6: now also GPIO46.1
- net at D47.2 (A), J19.A4 (VBUS), J19.A9 (VBUS)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: now also R155.2
- net at D44.2 (A), J11.A4 (VBUS), J11.A9 (VBUS)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: now also R78.2
- net GPIO3 renamed VBUS Detect USB1
- net VBUS Detect USB1: now also R153.1, R78.1
- net MCU2_GPIO3 renamed VBUS Detect USB2
- net VBUS Detect USB2: now also R154.1, R155.1
Other:
- note removed: "Rev #,Rbottom​ (Basic),Method,Ideal Vout​,ADC Count (12-bit),Window Range 00,Open Circuit,Internal Pull-up,~3.30V,4095,(Special Logic) 01,0Ω (Jumper),Grounded,0.00V,0,0 - 300 02,2.2kΩ,Divider,0.60V,739,301 - 1000 03,4.7kΩ,Divider,1.05V,1310,1001 - 1600 04,7.5kΩ,Divider,1.41V,1755,1601 - 2000 05,10kΩ,Divider,1.65V,2048,2001 - 2300 06,15kΩ,Divider,1.98V,2457,2301 - 2750 07,22kΩ,Divider,2.27V,2816,2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"
- moved on the sheet: D44, D47, R102, R103, R104, R105, R108, R109, R110, R111, R114, R115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
