File: CellKeeper/CellKeeper.kicad_pcb (KiCad board)
At the start: 4 copper layers, 260 x 113 mm, 470 parts, among them J1 Screw_Terminal_01x04, J10 3.81P Screw Terminal, J11 USB_C_Receptacle_USB2.0_16P, J12 Conn_02x10_Odd_Even, J14 ZE05H-8DP-2H, J15 Screw_Terminal_01x04, J16 Conn_01x03, J17 OEM HV Sense Connector, J18 7.62mm Pitch Screw Terminal, J19 USB_C_Receptacle_USB2.0_16P, J2 Screw_Terminal_01x01, J20 OEM Connector, J21 3.81P Screw Terminal, J22 Conn_02x10_Odd_Even, J3 Screw_Terminal_01x04, J4 8P8C_LED_Shielded_x2, J5 8P8C_LED_Shielded_x2, J6 S44B-RAD1AK, J7 Screw_Terminal_01x04, J8 Conn_01x03, J9 USB_C_Receptacle_USB2.0_16P, Q1 BSC0805LS, Q2 BSC0805LS, Q3 BSC0805LS, Q4 BSC0805LS, SW1 TS-1187A-B-A-B, SW2 TS-1187A-B-A-B, SW3 TS-1187A-B-A-B, SW4 TS-1187A-B-A-B, U1 UCC27524DR, U10 ISO1050DUB, U11 UCC27524DR, U12 LTV-217-B-G, U13 LTV-217-B-G, U14 RP2354B, U15 F0505S-1WR3, U16 ISO1540, U17 INA228, U18 ADS1115, U19 ADS1115, U20 RP2354B, U21 SP3485EN-L/TR, U22 AM26LV32EIDR, U25 TLV1117LV33DCYR, U26 TLV1117LV33DCYR, U3 TPS5430DDAR, U4 F0505S-1WR3, U5 ISO1050DUB, U6 LTV-217-B-G, U7 LTV-217-B-G, U8 LTV-217-B-G, U9 LTV-217-B-G, Y1 ABM8-272-T3, Y2 ABM8-272-T3

Commit message: Add 3D-printable enclosure for the main board (build123d)
enclosure/cellkeeper_case.py builds a base tray and lid around the board:
- M3 screws from below self-tap into the lid pillars at H1/H2/H7/H8 (and
  H3/H4 while BOARD_SCREWS_AT_H3_H4 is set); 45 deg screw seats print
  without support
- flat lid top 20 mm above the PCB with 4.3 mm bracket holes over H3/H4
  for the penthouse mounting brackets
- connector openings, J6 passing through the lid, ground-screw slot,
  button guide tubes and LED light tunnels
- lid markings as true curves: the silkscreen logo refit as lines and
  splines, KiBuzzard-style labels built from the KiBuzzard font
- print files as STEP/STL (whole and split for 256 mm beds), with
  separate inlay and light-pipe parts for multi-colour printing
- an interference check against the board's STEP export

Also:
- CellKeeper_Enclosure board-only footprint (ENC1 at 0,0) showing the
  case models in KiCad's 3D viewer
- recolor_vendor_step_models.py colours J20's terminals and hold-downs
  metal on the fused vendor solid
- board and schematic: current working changes, including the H7/H8
  mounting holes, the D34 move and the ENC1 enclosure footprint
Parts:
- added ENC1: CellKeeper_Enclosure, CellKeeper_Local:CellKeeper_Enclosure, F.Cu at (0.00, 0.00)
- added H7: MountingHole_Pad, CellKeeper_Local:MountingHole__MountingHole_3.7mm, F.Cu at (302.1, 137.5)
- added H8: MountingHole_Pad, CellKeeper_Local:MountingHole__MountingHole_3.7mm, F.Cu at (56.1, 137.5)
- added kibuzzard-6AD6CA76: G***, kibuzzard-6AD6CA76, F.Cu at (277.7, 131.7)
- moved R145 11.9 mm to (254.5, 136.7)
- moved JP37 5.92 mm to (271.5, 131.6), turned to 90 degrees
- moved D34 4.68 mm to (121.2, 81.1), turned to -90 degrees
- moved R146 0.10 mm to (254.5, 130.7)
Routing:
- net Net-(R145-Pad1): track 13.3 -> 3.08 mm
- net Net-(C19-Pad1): track 63.3 -> 72.0 mm, vias 1 -> 2
- net Net-(D34-A): track 1.54 -> 6.41 mm
- net GND: track 249.6 -> 252.7 mm, vias 158 -> 157
- net GND CAN: track 31.9 -> 34.7 mm
- net Net-(J4-Pad18): track 36.6 -> 35.9 mm
Other:
- board text added: "13-16V"
- board text removed: "12-16V"
- board text removed: "E-STOP"
